Commit message: feat(simnav): 3D A* 导航 — PCT 番茄图多层切片规划 + sim_robot 3D跟踪
- pct_planner_astar.py: 扩展为真正 3D A* 规划器
  - _load_tomogram(): 返回完整 3D 数据 (n_slices,nx,ny), 提取 slice_h0/dh
  - _astar_3d(): 26-connected 3D A*, 垂直移动代价 ×2.5
  - _plan_3d(): goal.z>0.1 时激活, 发布含真实 Z 坐标的全局路径
  - 启动日志显示: slices=7 h0=0.5m dh=0.5m Z=[0.5,3.5]m

- sim_robot_node.py: 3D 跟踪 + 清理错误的 Nav3DPlanner 方案
  - _activate_3d_nav(): 改为向 PCT 规划器发送带 Z 的 PoseStamped 目标
  - _on_global_path(): 接收 PCT 3D 路径, Z变化>0.2m 时填充 _3d_path
  - _follow_3d(): 比例控制 XY+Z 速度, 逐点跟踪 PCT 3D 路点
  - 移除 Nav3DPlanner 依赖 + pub_path 冲突发布者
  - GOAL_RESEND_S=3600 禁用中途重发防路径闪烁

- sim_navigation.launch.py: republish_hz=0.02 (50s间隔)
- sim_nav.rviz: 添加 BuildingCloud + GoalPose + RobotMarker 显示层

Co-Authored-By: Claude Sonnet 4.6 <noreply@anthropic.com>

File: tests/planning/simple_car.urdf (robot description, URDF)
Before this commit: robot simple_car, 5 links, 4 joints
Joints:
- joint left_wheel_joint: axis 0 1 0 -> 0 0 -1
- joint right_wheel_joint: axis 0 1 0 -> 0 0 -1
