Commit message: refactor: sim/robot — Thunder 产品 URDF 替代旧模型
- 新增 thunder.urdf (轮足狗机器人v3, 18.69kg, 16DOF+4轮)
- 删除 dog_arm.urdf / robot.xml (旧模型)
- .gitignore 排除 STL mesh 二进制

Co-Authored-By: Claude Opus 4.6 (1M context) <noreply@anthropic.com>

File: sim/robot/thunder.urdf (robot description, URDF)
Before this commit: robot dog_arm, 30 links, 29 joints
Links:
- removed link arm_gripper_left
- removed link arm_gripper_right
- removed link arm_link_0
- removed link arm_link_1
- removed link arm_link_2
- removed link arm_link_3
- removed link arm_link_4
- removed link arm_link_5
- removed link arm_link_6
- link base_link: geometry collision box size=0.05 0.27 0.14; collision box size=0.05 0.27 0.14
- link camera1_Link: geometry visual mesh filename=thunder_meshes/camera1_Link.STL
- link camera2_Link: geometry visual mesh filename=thunder_meshes/camera2_Link.STL
- link fl_calf_Link: geometry collision box size=0.18 0.04 0.045; collision cylinder length=0.03 radius=0.0635
- link fl_foot_Link: geometry collision cylinder length=0.05617 radius=0.12; visual mesh filename=thunder_meshes/fl_foot_Link.STL
- link fl_hip_Link: mass 1.66356 -> 1.78126; geometry collision cylinder length=0.048 radius=0.06; visual mesh filename=thunder_meshes/fl_hip_Link.STL
- link fl_thigh_Link: mass 2.41000 -> 2.40982; geometry collision box size=0.18 0.03 0.06; collision cylinder length=0.03 radius=0.064
- link fr_calf_Link: geometry collision box size=0.18 0.04 0.045; collision cylinder length=0.03 radius=0.0635
- link fr_foot_Link: geometry collision cylinder length=0.05617 radius=0.12; visual mesh filename=thunder_meshes/fr_foot_Link.STL
- link fr_hip_Link: mass 1.66356 -> 1.78126; geometry collision cylinder length=0.048 radius=0.06; visual mesh filename=thunder_meshes/fr_hip_Link.STL
- link fr_thigh_Link: mass 2.41000 -> 2.40982; geometry collision box size=0.18 0.03 0.06; collision cylinder length=0.03 radius=0.064
- link lidar1_Link: geometry visual mesh filename=thunder_meshes/lidar1_Link.STL
- link lidar2_Link: geometry collision box size=0.0768 0.0768 0.0801; visual mesh filename=thunder_meshes/lidar2_Link.STL
- link rl_calf_Link: geometry collision box size=0.18 0.04 0.045; collision cylinder length=0.03 radius=0.0635
- link rl_foot_Link: geometry collision cylinder length=0.05617 radius=0.12; visual mesh filename=thunder_meshes/rl_foot_Link.STL
- link rl_hip_Link: mass 1.66356 -> 1.78126; geometry collision cylinder length=0.048 radius=0.06; visual mesh filename=thunder_meshes/rl_hip_Link.STL
- link rl_thigh_Link: mass 2.41000 -> 2.40982; geometry collision box size=0.18 0.03 0.06; collision cylinder length=0.03 radius=0.064
- link rr_calf_Link: geometry collision box size=0.18 0.04 0.045; collision cylinder length=0.03 radius=0.0635
- link rr_foot_Link: geometry collision cylinder length=0.05617 radius=0.12; visual mesh filename=thunder_meshes/rr_foot_Link.STL
- link rr_hip_Link: mass 1.66356 -> 1.78126; geometry collision cylinder length=0.048 radius=0.06; visual mesh filename=thunder_meshes/rr_hip_Link.STL
- link rr_thigh_Link: mass 2.41000 -> 2.40982; geometry collision box size=0.18 0.03 0.06; collision cylinder length=0.03 radius=0.064
Joints:
- removed joint arm_gripper_left_joint
- removed joint arm_gripper_right_joint
- removed joint arm_joint_1
- removed joint arm_joint_2
- removed joint arm_joint_3
- removed joint arm_joint_4
- removed joint arm_joint_5
- removed joint arm_joint_6
- removed joint base_to_arm_joint
- joint camera2_joint: axis 0 0.012973 0.99992 -> (none); limit lower=0 upper=0 effort=0 velocity=0 -> (none)
- joint fl_foot_joint: type revolute -> continuous
- joint fl_hip_joint: origin xyz=0.2395 0.065405 0.08065 rpy=0 0 0 -> xyz=0.2395 0.065 0.08065 rpy=0 0 0
- joint fr_foot_joint: type revolute -> continuous
- joint fr_hip_joint: origin xyz=0.2395 -0.064595 0.08065 rpy=0 0 0 -> xyz=0.2395 -0.065 0.08065 rpy=0 0 0
- joint rl_foot_joint: type revolute -> continuous
- joint rl_hip_joint: origin xyz=-0.2395 0.063755 0.08065 rpy=0 0 0 -> xyz=-0.2395 0.065 0.08065 rpy=0 0 0
- joint rr_calf_joint: axis 0 0.99997 0.0079551 -> 0 1 0; origin xyz=0.24946 -0.056867 -0.016903 rpy=0 0 0 -> xyz=0.24954 -0.057 -0.01515 rpy=0 0 0
- joint rr_foot_joint: axis 0 0.99997 0.0079551 -> 0 1 0; origin xyz=-0.24377 -0.061439 0.054994 rpy=0 0 0 -> xyz=-0.24443 -0.061 0.0525 rpy=0 0 0; type revolute -> continuous
- joint rr_hip_joint: origin xyz=-0.2395 -0.066245 0.08065 rpy=0 0 0 -> xyz=-0.2395 -0.065 0.08065 rpy=0 0 0
- joint rr_thigh_joint: axis 0 0.99997 0.0079551 -> 0 1 0; origin xyz=-0.078 -0.079497 -0.00063243 rpy=0 0 0 -> xyz=-0.078 -0.0795 0 rpy=0 0 0

Commit message: refactor(sim): thunder URDF 命名标准化 + mesh 目录迁移
- robot name: 中文 "轮足狗机器人v3" → "wheeled_legged_dog_v3"（避免
  ROS2/MuJoCo/Isaac Lab 在不同 locale 下解析报错）
- link 命名: fr_hip_Link → FR_hip 等（统一 Isaac Lab/MuJoCo RL 训练
  侧使用的 SCREAMING 前缀 + 去掉 _Link 后缀）
- mesh 路径: thunder_meshes/X.STL → ../meshes/X.STL，把 21 个 STL 从
  sim/robot/thunder_meshes/ 物理移到 sim/meshes/，同步 .gitignore

实际 STL 文件仍然不进 git（保留 LFS-or-external 约定），但 ignore
规则从 sim/robot/.gitignore 迁到 sim/meshes/.gitignore，跟 URDF 引用
路径保持一致。

Co-Authored-By: Claude Opus 4.7 (1M context) <noreply@anthropic.com>

File: sim/robot/thunder.urdf (robot description, URDF)
Before this commit: robot 轮足狗机器人v3, 21 links, 20 joints
Links:
- removed link fl_calf_Link
- removed link fl_foot_Link
- removed link fl_hip_Link
- removed link fl_thigh_Link
- removed link fr_calf_Link
- removed link fr_foot_Link
- removed link fr_hip_Link
- removed link fr_thigh_Link
- removed link rl_calf_Link
- removed link rl_foot_Link
- removed link rl_hip_Link
- removed link rl_thigh_Link
- removed link rr_calf_Link
- removed link rr_foot_Link
- removed link rr_hip_Link
- removed link rr_thigh_Link
- added link FL_calf, mass 1.89384; collision box size=0.18 0.04 0.045; collision cylinder length=0.03 radius=0.0635
- added link FL_foot, mass 0.32377; collision cylinder length=0.05617 radius=0.12; visual mesh filename=../meshes/fl_foot_Link.STL
- added link FL_hip, mass 1.78126; collision cylinder length=0.048 radius=0.06; visual mesh filename=../meshes/fl_hip_Link.STL
- added link FL_thigh, mass 2.40982; collision box size=0.18 0.03 0.06; collision cylinder length=0.03 radius=0.064
- added link FR_calf, mass 1.89384; collision box size=0.18 0.04 0.045; collision cylinder length=0.03 radius=0.0635
- added link FR_foot, mass 0.32377; collision cylinder length=0.05617 radius=0.12; visual mesh filename=../meshes/fr_foot_Link.STL
- added link FR_hip, mass 1.78126; collision cylinder length=0.048 radius=0.06; visual mesh filename=../meshes/fr_hip_Link.STL
- added link FR_thigh, mass 2.40982; collision box size=0.18 0.03 0.06; collision cylinder length=0.03 radius=0.064
- added link RL_calf, mass 1.89384; collision box size=0.18 0.04 0.045; collision cylinder length=0.03 radius=0.0635
- added link RL_foot, mass 0.32377; collision cylinder length=0.05617 radius=0.12; visual mesh filename=../meshes/rl_foot_Link.STL
- added link RL_hip, mass 1.78126; collision cylinder length=0.048 radius=0.06; visual mesh filename=../meshes/rl_hip_Link.STL
- added link RL_thigh, mass 2.40982; collision box size=0.18 0.03 0.06; collision cylinder length=0.03 radius=0.064
- added link RR_calf, mass 1.89384; collision box size=0.18 0.04 0.045; collision cylinder length=0.03 radius=0.0635
- added link RR_foot, mass 0.32377; collision cylinder length=0.05617 radius=0.12; visual mesh filename=../meshes/rr_foot_Link.STL
- added link RR_hip, mass 1.78126; collision cylinder length=0.048 radius=0.06; visual mesh filename=../meshes/rr_hip_Link.STL
- added link RR_thigh, mass 2.40982; collision box size=0.18 0.03 0.06; collision cylinder length=0.03 radius=0.064
- link base_link: geometry collision box size=0.05 0.27 0.14; collision box size=0.05 0.27 0.14
- link camera1_Link: geometry visual mesh filename=../meshes/camera1_Link.STL
- link camera2_Link: geometry visual mesh filename=../meshes/camera2_Link.STL
- link lidar1_Link: geometry visual mesh filename=../meshes/lidar1_Link.STL
- link lidar2_Link: geometry collision box size=0.0768 0.0768 0.0801; visual mesh filename=../meshes/lidar2_Link.STL
Joints:
- joint fl_calf_joint: child fl_calf_Link -> FL_calf; parent fl_thigh_Link -> FL_thigh
- joint fl_foot_joint: child fl_foot_Link -> FL_foot; parent fl_calf_Link -> FL_calf
- joint fl_hip_joint: child fl_hip_Link -> FL_hip
- joint fl_thigh_joint: child fl_thigh_Link -> FL_thigh; parent fl_hip_Link -> FL_hip
- joint fr_calf_joint: child fr_calf_Link -> FR_calf; parent fr_thigh_Link -> FR_thigh
- joint fr_foot_joint: child fr_foot_Link -> FR_foot; parent fr_calf_Link -> FR_calf
- joint fr_hip_joint: child fr_hip_Link -> FR_hip
- joint fr_thigh_joint: child fr_thigh_Link -> FR_thigh; parent fr_hip_Link -> FR_hip
- joint rl_calf_joint: child rl_calf_Link -> RL_calf; parent rl_thigh_Link -> RL_thigh
- joint rl_foot_joint: child rl_foot_Link -> RL_foot; parent rl_calf_Link -> RL_calf
- joint rl_hip_joint: child rl_hip_Link -> RL_hip
- joint rl_thigh_joint: child rl_thigh_Link -> RL_thigh; parent rl_hip_Link -> RL_hip
- joint rr_calf_joint: child rr_calf_Link -> RR_calf; parent rr_thigh_Link -> RR_thigh
- joint rr_foot_joint: child rr_foot_Link -> RR_foot; parent rr_calf_Link -> RR_calf
- joint rr_hip_joint: child rr_hip_Link -> RR_hip
- joint rr_thigh_joint: child rr_thigh_Link -> RR_thigh; parent rr_hip_Link -> RR_hip
