Commit message: Preserve navigation validation while upgrading Thunder simulation
The route validation tooling, exploration wiring, and Thunder v3 simulation assets move the robot stack toward a safer upgrade path without changing the deployed control chain. Routecheck keeps plan validation non-motion by default, while the simulator now follows the current Thunder v3 geometry and actuator naming through compatibility adapters.

Constraint: Real-robot verification must remain non-motion; no goal, teleop, or cmd_vel commands were sent.

Constraint: Existing localization/nav service ownership stays external via localizer bridge.

Rejected: Switch nav back to managed FastLIO | would change the robot runtime ownership model and risk service conflicts.

Rejected: Commit generated pycache/status artifacts | not source of truth and not needed for runtime.

Confidence: high

Scope-risk: moderate

Directive: Keep routecheck non-motion by default; routecompare must stay behind explicit --allow-motion and should not be used during readiness checks.

Tested: python -m pytest src/core/tests/ -q --tb=short (2019 passed, 7 skipped)

Tested: deployment/sim/Gateway/calibration/profile/SLAM focused pytest suites

Tested: bash -n scripts/lingtu

Tested: robot /ready and /api/v1/app/bootstrap read-only checks

Tested: robot scripts/lingtu soak --duration 15 --interval 5 --json --strict

Not-tested: Real routecompare motion run; camera video frames remain unavailable because Orbbec is not enumerated by Linux.

File: sim/assets/urdf/thunder_v3.urdf (robot description, URDF)
Before this commit: robot thunder_v3, 21 links, 20 joints
Links:
- link FL_calf: geometry collision box size=0.18 0.04 0.045; collision cylinder length=0.03 radius=0.0635
- link FL_foot: geometry collision cylinder length=0.05617 radius=0.12; visual mesh filename=../meshes/fl_foot_Link.STL
- link FL_hip: geometry collision cylinder length=0.048 radius=0.06; visual mesh filename=../meshes/fl_hip_Link.STL
- link FL_thigh: geometry collision box size=0.18 0.03 0.06; collision cylinder length=0.03 radius=0.064
- link FR_calf: geometry collision box size=0.18 0.04 0.045; collision cylinder length=0.03 radius=0.0635
- link FR_foot: geometry collision cylinder length=0.05617 radius=0.12; visual mesh filename=../meshes/fr_foot_Link.STL
- link FR_hip: geometry collision cylinder length=0.048 radius=0.06; visual mesh filename=../meshes/fr_hip_Link.STL
- link FR_thigh: geometry collision box size=0.18 0.03 0.06; collision cylinder length=0.03 radius=0.064
- link RL_calf: geometry collision box size=0.18 0.04 0.045; collision cylinder length=0.03 radius=0.0635
- link RL_foot: geometry collision cylinder length=0.05617 radius=0.12; visual mesh filename=../meshes/rl_foot_Link.STL
- link RL_hip: geometry collision cylinder length=0.048 radius=0.06; visual mesh filename=../meshes/rl_hip_Link.STL
- link RL_thigh: geometry collision box size=0.18 0.03 0.06; collision cylinder length=0.03 radius=0.064
- link RR_calf: geometry collision box size=0.18 0.04 0.045; collision cylinder length=0.03 radius=0.0635
- link RR_foot: geometry collision cylinder length=0.05617 radius=0.12; visual mesh filename=../meshes/rr_foot_Link.STL
- link RR_hip: geometry collision cylinder length=0.048 radius=0.06; visual mesh filename=../meshes/rr_hip_Link.STL
- link RR_thigh: geometry collision box size=0.18 0.03 0.06; collision cylinder length=0.03 radius=0.064
- link base_link: geometry collision box size=0.05 0.27 0.14; collision box size=0.05 0.27 0.14
- link camera1_Link: geometry visual mesh filename=../meshes/camera1_Link.STL
- link camera2_Link: geometry visual mesh filename=../meshes/camera2_Link.STL
- link lidar1_Link: geometry visual mesh filename=../meshes/lidar1_Link.STL
- link lidar2_Link: geometry collision box size=0.0768 0.0768 0.0801; visual mesh filename=../meshes/lidar2_Link.STL
